Commit message: Update for kinetic and various cleanup

File: std_parts.xacro (robot description, xacro)
@@ -5,54 +5,54 @@
     <link name="torso_link">
         <visual>
-            <xacro:default_geometry cad_file="BPF-CHEST-F"/>
+            <default_geometry cad_file="BPF-CHEST-F"/>
             <origin rpy="${pi/2} 0 ${pi/2}"/>
         </visual>
         <visual>
-            <xacro:default_geometry cad_file="BPF-CHEST-B"/>
+            <default_geometry cad_file="BPF-CHEST-B"/>
             <origin rpy="${pi/2} 0 ${pi/2}"/>
         </visual>
         <visual>
-            <xacro:default_geometry cad_file="CM-5"/>
+            <default_geometry cad_file="CM-5"/>
             <origin xyz="-0.032 0 -0.015" rpy="0 ${pi} ${pi/2}"/>
         </visual>
         <!-- Sensor 100 -->
         <visual>
-            <xacro:default_geometry cad_file="AX-S1"/>
+            <default_geometry cad_file="AX-S1"/>
             <origin xyz="0 0 0.025" rpy="${-pi/2} 0 ${-pi/2}"/>
         </visual>
         <!-- Motor 1 -->
         <visual>
-            <xacro:default_geometry cad_file="AX-12"/>
+            <default_geometry cad_file="AX-12"/>
             <origin xyz="0 -0.032 0" rpy="${pi/2} 0 0"/>
         </visual>
         <visual>
-            <xacro:default_geometry cad_file="FP04-F3"/>
+            <default_geometry cad_file="FP04-F3"/>
             <origin xyz="-0.019 -0.032 -0.0145" rpy="${pi} ${-pi/2} ${pi/2}"/>
         </visual>
         <!-- Motor 2 -->
         <visual>
-            <xacro:default_geometry cad_file="AX-12"/>
+            <default_geometry cad_file="AX-12"/>
             <origin xyz="0 0.032 0" rpy="${pi/2} 0 ${pi}"/>
         </visual>
         <visual>
-            <xacro:default_geometry cad_file="FP04-F3"/>
+            <default_geometry cad_file="FP04-F3"/>
             <origin xyz="-0.019 0.032 -0.0145" rpy="${pi} ${-pi/2} ${pi/2}"/>
         </visual>
         <visual>
-            <xacro:default_geometry cad_file="FP04-F3"/>
+            <default_geometry cad_file="FP04-F3"/>
             <origin xyz="0.0175 0 -0.0655" rpy="0 0 ${pi/2}"/>
         </visual>
         <visual>
-            <xacro:default_geometry cad_file="FP04-F3"/>
+            <default_geometry cad_file="FP04-F3"/>
             <origin xyz="-0.0175 0 -0.0655" rpy="0 0 ${-pi/2}"/>
         </visual>
         <!-- Motor 7 -->
         <visual>
-            <xacro:default_geometry cad_file="AX-12"/>
+            <default_geometry cad_file="AX-12"/>
             <origin xyz="0 -0.0385 -0.0655" rpy="0 ${pi} ${pi}"/>
         </visual>
         <!-- Motor 8 -->
         <visual>
-            <xacro:default_geometry cad_file="AX-12"/>
+            <default_geometry cad_file="AX-12"/>
             <origin xyz="0 0.0385 -0.0655" rpy="0 ${pi} 0"/>
         </visual>
@@ -84,5 +84,5 @@
     <link name="r_foot_link">
         <visual>
-            <xacro:default_geometry cad_file="FP04-F12"/>
+            <default_geometry cad_file="FP04-F12"/>
             <origin xyz="0.0235 0 0" rpy="0 ${pi/2} ${-pi/2}"/>
         </visual>
@@ -102,5 +102,5 @@
     <link name="l_foot_link">
         <visual>
-            <xacro:default_geometry cad_file="FP04-F12"/>
+            <default_geometry cad_file="FP04-F12"/>
             <origin xyz="-0.0235 0 0" rpy="${pi} ${pi/2} ${-pi/2}"/>
         </visual>

File: typea.urdf (robot description, URDF)
Before this commit: robot typea, 24 links, 23 joints
Links:
- added link imu_link; visual box size=0.04 0.02 0.005
- link l_ankle_lateral_link: geometry collision box size=0.0405 0.029 0.083; visual mesh filename=file:///home/mathieu/work/ros-kinetic/my-bioloid/src/bioloi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 scale=0.001 0.001 0.001
- link l_ankle_swing_link: geometry collision box size=0.051 0.0721 0.04; visual mesh filename=file:///home/mathieu/work/ros-kinetic/my-bioloid/src/bioloi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 scale=0.001 0.001 0.001
- link l_foot_link: geometry collision box size=0.009 0.061 0.101; visual mesh filename=file:///home/mathieu/work/ros-kinetic/my-bioloid/src/bioloi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 scale=0.001 0.001 0.001
- link l_hand_link: geometry collision box size=0.0131 0.0265 0.044; collision box size=0.0575 0.0175 0.035
- link l_hip_lateral_link: geometry collision box size=0.04 0.051 0.0721; visual mesh filename=file:///home/mathieu/work/ros-kinetic/my-bioloid/src/bioloi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 scale=0.001 0.001 0.001
- link l_hip_twist_link: geometry collision box size=0.029 0.083 0.0405; visual mesh filename=file:///home/mathieu/work/ros-kinetic/my-bioloid/src/bioloi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 scale=0.001 0.001 0.001
- link l_lower_arm_link: geometry collision box size=0.058 0.033 0.044; visual mesh filename=file:///home/mathieu/work/ros-kinetic/my-bioloid/src/bioloi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 scale=0.001 0.001 0.001
- link l_lower_leg_link: geometry collision box size=0.033 0.051 0.044; collision box size=0.067 0.03 0.049
- link l_shoulder_swing_link: geometry collision box size=0.052 0.039 0.036; visual mesh filename=file:///home/mathieu/work/ros-kinetic/my-bioloid/src/bioloi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 scale=0.001 0.001 0.001
- link l_upper_arm_link: geometry collision box size=0.047 0.033 0.052; collision box size=0.054 0.033 0.044
- link l_upper_leg_link: geometry collision box size=0.04 0.0371 0.049; collision box size=0.065 0.03 0.049
- link r_ankle_lateral_link: geometry collision box size=0.0405 0.029 0.083; visual mesh filename=file:///home/mathieu/work/ros-kinetic/my-bioloid/src/bioloi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 scale=0.001 0.001 0.001
- link r_ankle_swing_link: geometry collision box size=0.051 0.0721 0.04; visual mesh filename=file:///home/mathieu/work/ros-kinetic/my-bioloid/src/bioloi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 scale=0.001 0.001 0.001
- link r_foot_link: geometry collision box size=0.009 0.061 0.101; visual mesh filename=file:///home/mathieu/work/ros-kinetic/my-bioloid/src/bioloi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 scale=0.001 0.001 0.001
- link r_hand_link: geometry collision box size=0.0131 0.0265 0.044; collision box size=0.0575 0.0175 0.035
- link r_hip_lateral_link: geometry collision box size=0.04 0.051 0.0721; visual mesh filename=file:///home/mathieu/work/ros-kinetic/my-bioloid/src/bioloi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 scale=0.001 0.001 0.001
- link r_hip_twist_link: geometry collision box size=0.029 0.083 0.0405; visual mesh filename=file:///home/mathieu/work/ros-kinetic/my-bioloid/src/bioloi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 scale=0.001 0.001 0.001
- link r_lower_arm_link: geometry collision box size=0.058 0.033 0.044; visual mesh filename=file:///home/mathieu/work/ros-kinetic/my-bioloid/src/bioloi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 scale=0.001 0.001 0.001
- link r_lower_leg_link: geometry collision box size=0.033 0.051 0.044; collision box size=0.067 0.03 0.049
- link r_shoulder_swing_link: geometry collision box size=0.052 0.039 0.036; visual mesh filename=file:///home/mathieu/work/ros-kinetic/my-bioloid/src/bioloi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 scale=0.001 0.001 0.001
- link r_upper_arm_link: geometry collision box size=0.047 0.033 0.052; collision box size=0.054 0.033 0.044
- link r_upper_leg_link: geometry collision box size=0.04 0.0371 0.049; collision box size=0.065 0.03 0.049
- link torso_link: geometry collision box size=0.054 0.033 0.044; collision box size=0.065 0.099 0.043
Joints:
- added joint imu_to_base_joint: type fixed, parent imu_link, child base_link, origin xyz=0.01 0 0.0788 rpy=0 0 0
- joint l_ankle_lateral_joint: limit lower=-2.61799166667 upper=2.61799166667 effort=10 velocity=5.6548668 -> lower=-0.5 upper=0.5 effort=10 velocity=5.6548668
- joint l_ankle_swing_joint: limit lower=-2.61799166667 upper=2.61799166667 effort=10 velocity=5.6548668 -> lower=-1.0 upper=0.4 effort=10 velocity=5.6548668
- joint l_hip_lateral_joint: limit lower=-2.61799166667 upper=2.61799166667 effort=10 velocity=5.6548668 -> lower=-0.6 upper=0.6 effort=10 velocity=5.6548668
- joint l_hip_swing_joint: limit lower=-2.61799166667 upper=2.61799166667 effort=10 velocity=5.6548668 -> lower=-0.4 upper=1.0 effort=10 velocity=5.6548668
- joint l_hip_twist_joint: limit lower=-2.61799166667 upper=2.61799166667 effort=10 velocity=5.6548668 -> lower=-0.5 upper=0.5 effort=10 velocity=5.6548668
- joint l_knee_joint: axis 0 0 1 -> 0 0 -1; limit lower=-2.61799166667 upper=2.61799166667 effort=10 velocity=5.6548668 -> lower=-0.0 upper=1.1 effort=10 velocity=5.6548668
- joint l_shoulder_lateral_joint: limit lower=-3.14159 upper=3.14159 effort=2.8 velocity=1.0 -> lower=-1.5 upper=1.5 effort=2.8 velocity=1.0
- joint l_shoulder_swing_joint: limit lower=-3.14159 upper=3.14159 effort=2.8 velocity=1.0 -> lower=-1 upper=1.570795 effort=2.8 velocity=1.0
- joint r_ankle_lateral_joint: limit lower=-2.61799166667 upper=2.61799166667 effort=10 velocity=5.6548668 -> lower=-0.5 upper=0.5 effort=10 velocity=5.6548668
- joint r_ankle_swing_joint: limit lower=-2.61799166667 upper=2.61799166667 effort=10 velocity=5.6548668 -> lower=-0.4 upper=1.0 effort=10 velocity=5.6548668
- joint r_hip_lateral_joint: limit lower=-2.61799166667 upper=2.61799166667 effort=10 velocity=5.6548668 -> lower=-0.6 upper=0.6 effort=10 velocity=5.6548668
- joint r_hip_swing_joint: limit lower=-2.61799166667 upper=2.61799166667 effort=10 velocity=5.6548668 -> lower=-1.0 upper=0.4 effort=10 velocity=5.6548668
- joint r_hip_twist_joint: limit lower=-2.61799166667 upper=2.61799166667 effort=10 velocity=5.6548668 -> lower=-0.5 upper=0.5 effort=10 velocity=5.6548668
- joint r_knee_joint: axis 0 0 1 -> 0 0 -1; limit lower=-2.61799166667 upper=2.61799166667 effort=10 velocity=5.6548668 -> lower=-1.1 upper=-0.0 effort=10 velocity=5.6548668
- joint r_shoulder_lateral_joint: limit lower=-3.14159 upper=3.14159 effort=2.8 velocity=1.0 -> lower=-1.5 upper=1.5 effort=2.8 velocity=1.0
- joint r_shoulder_swing_joint: limit lower=-3.14159 upper=3.14159 effort=2.8 velocity=1.0 -> lower=-1 upper=1.570795 effort=2.8 velocity=1.0
