Commit message: Update for kinetic and various cleanup

File: typea.xacro (robot description, xacro)
@@ -1,7 +1,4 @@
 <?xml version="1.0"?>
 <robot xmlns:xacro="http://www.ros.org/wiki/xacro" name="typea">
-    <!-- Standard parts of Bioloid Comprehensive humanoid with 18 AX-12+ servos, which have been replaced in custom version -->
-    <!--  When using this URDF, ensure a transform from odom to base_link is being published -->
-    <xacro:include filename="$(find bioloid_typea_description)/std_parts.xacro" ns="std_parts"/>
     <!-- Import gazebo_ros_control plugin -->
     <xacro:include filename="$(find bioloid_typea_description)/gazebo.xacro" ns="gazebo"/>
@@ -14,7 +11,32 @@
         </geometry>
     </xacro:macro>
-    <xacro:macro name="z_rot">
+    <xacro:macro name="xacro:z_rot">
         <axis xyz="0 0 1"/>
     </xacro:macro>
+    <!-- Standard parts of Bioloid Comprehensive humanoid with 18 AX-12+ servos, which have been replaced in custom version -->
+    <!--  When using this URDF, ensure a transform from odom to base_link is being published -->
+    <!-- <xacro:include filename="$(find bioloid_typea_description)/std_parts.xacro" ns="std_parts"/> -->
+    <xacro:include filename="$(find bioloid_typea_description)/std_parts.xacro"/>
+    <!-- IMU -->
+    <joint name="imu_to_base_joint" type="fixed">
+        <parent link="imu_link"/>
+        <origin xyz="0.01 0 0.0788" rpy="0 0 0"/>
+        <child link="base_link"/>
+    </joint>
+    <link name="imu_link">
+        <visual>
+            <geometry>
+                <box size="0.04 0.02 0.005"/>
+            </geometry>
+            <material name="green">
+                <color rgba="0.0 1.0 0.0 1.0"/>
+            </material>
+        </visual>
+        <!--<inertial>
+            <origin xyz="0 0 0"/>
+            <mass value="1.0"/>
+            <inertia  ixx="0.001" ixy="0.0"  ixz="0.0"  iyy="0.001"  iyz="0.0"  izz="0.001"/>
+        </inertial>-->
+    </link>
     <xacro:macro name="shoulder_swing_joint" params="prefix reflect">
         <joint name="${prefix}_shoulder_swing_joint" type="revolute">
@@ -23,5 +45,5 @@
             <xacro:z_rot/>
             <child link="${prefix}_shoulder_swing_link"/>
-            <limit lower="${-pi}" upper="${pi}" effort="2.8" velocity="1.0"/>
+            <limit lower="-1" upper="${pi/2}" effort="2.8" velocity="1.0"/>
         </joint>
     </xacro:macro>
@@ -32,5 +54,5 @@
             <xacro:z_rot/>
             <child link="${prefix}_upper_arm_link"/>
-            <limit lower="${-pi}" upper="${pi}" effort="2.8" velocity="1.0"/>
+            <limit lower="-1.5" upper="1.5" effort="2.8" velocity="1.0"/>
         </joint>
     </xacro:macro>
@@ -41,5 +63,5 @@
             <xacro:z_rot/>
             <child link="${prefix}_lower_arm_link"/>
-            <limit lower="${-1.77}" upper="${1.77}" effort="2.8" velocity="1.0"/>
+            <limit lower="-1.77" upper="1.77" effort="2.8" velocity="1.0"/>
         </joint>
     </xacro:macro>
@@ -57,5 +79,5 @@
             <xacro:z_rot/>
             <child link="${prefix}_hip_twist_link"/>
-            <limit lower="${-pi*5/6}" upper="${pi*5/6}" effort="10" velocity="5.6548668"/>
+            <limit lower="-0.5" upper="0.5" effort="10" velocity="5.6548668"/>
         </joint>
     </xacro:macro>
@@ -66,5 +88,5 @@
             <xacro:z_rot/>
             <child link="${prefix}_hip_lateral_link"/>
-            <limit lower="${-pi*5/6}" upper="${pi*5/6}" effort="10" velocity="5.6548668"/>
+            <limit lower="-0.6" upper="0.6" effort="10" velocity="5.6548668"/>
         </joint>
     </xacro:macro>
@@ -75,5 +97,5 @@
             <xacro:z_rot/>
             <child link="${prefix}_upper_leg_link"/>
-            <limit lower="${-pi*5/6}" upper="${pi*5/6}" effort="10" velocity="5.6548668"/>
+            <limit lower="${-0.3*(reflect-1)-1}" upper="${-0.3*(reflect+1)+1}" effort="10" velocity="5.6548668"/>
         </joint>
     </xacro:macro>
@@ -82,7 +104,7 @@
             <parent link="${prefix}_upper_leg_link"/>
             <origin xyz="${reflect*0.075} 0.0145 0" rpy="0 0 0"/>
-            <xacro:z_rot/>
+            <axis xyz="0 0 -1"/>
             <child link="${prefix}_lower_leg_link"/>
-            <limit lower="${-pi*5/6}" upper="${pi*5/6}" effort="10" velocity="5.6548668"/>
+            <limit lower="${-0.55*(1+reflect)}" upper="${-0.55*(-1+reflect)}" effort="10" velocity="5.6548668"/>
         </joint>
     </xacro:macro>
@@ -93,5 +115,5 @@
             <xacro:z_rot/>
             <child link="${prefix}_ankle_swing_link"/>
-            <limit lower="${-pi*5/6}" upper="${pi*5/6}" effort="10" velocity="5.6548668"/>
+            <limit lower="${0.3*(reflect+1)-1}" upper="${0.3*(reflect-1)+1}" effort="10" velocity="5.6548668"/>
         </joint>
     </xacro:macro>
@@ -102,5 +124,5 @@
             <xacro:z_rot/>
             <child link="${prefix}_ankle_lateral_link"/>
-            <limit lower="${-pi*5/6}" upper="${pi*5/6}" effort="10" velocity="5.6548668"/>
+            <limit lower="-0.5" upper="0.5" effort="10" velocity="5.6548668"/>
         </joint>
     </xacro:macro>
@@ -125,26 +147,26 @@
         <!-- Motor 9[r] 10[l] -->
         <visual>
-            <xacro:default_geometry cad_file="AX-12"/>
+            <default_geometry cad_file="AX-12"/>
             <origin xyz="0 0 ${z_offset}" rpy="0 0 ${(reflect-1)*pi*-1/2}"/>
         </visual>
         <visual>
-            <xacro:default_geometry cad_file="FP04-F6"/>
+            <default_geometry cad_file="FP04-F6"/>
             <origin xyz="${-1*reflect*0.019} ${-1*reflect*0.0145} ${z_offset+0.016}" rpy="0 ${-pi/2} ${-1*reflect*pi/2}"/>
         </visual>
         <visual>
-            <xacro:default_geometry cad_file="FP04-F6"/>
+            <default_geometry cad_file="FP04-F6"/>
             <origin xyz="${reflect*0.019} ${-1*reflect*0.0145} ${z_offset+0.016}" rpy="0 ${-pi/2} ${reflect*pi/2}"/>
         </visual>
         <!-- Motor 11[r] 12[l] -->
         <visual>
-            <xacro:default_geometry cad_file="AX-12"/>
+            <default_geometry cad_file="AX-12"/>
             <origin xyz="0 0 ${z_offset-0.032}" rpy="${(reflect-1)*pi*-1/2} ${-1*reflect*pi/2} 0"/>
         </visual>
         <visual>
-            <xacro:default_geometry cad_file="BPF-BU"/>
+            <default_geometry cad_file="BPF-BU"/>
             <origin xyz="0 0 ${z_offset-0.05}" rpy="${-1*reflect*pi/2} ${(reflect-1)*pi*-1/2} 0"/>
         </visual>
         <visual>
-            <xacro:default_geometry cad_file="FP04-F7"/>
+            <default_geometry cad_file="FP04-F7"/>
             <origin xyz="0 ${-1*reflect*0.0145} ${z_offset-0.051}" rpy="${reflect*pi/2} ${(reflect-1)*pi*-1/2} ${pi/2}"/>
         </visual>
@@ -165,5 +187,5 @@
     <link name="${prefix}_hip_twist_link">
         <visual>
-            <xacro:default_geometry cad_file="FP04-F5"/>
+            <default_geometry cad_file="FP04-F5"/>
             <origin xyz="0 ${reflect*y_offset} 0.05" rpy="${pi} 0 ${(reflect+1)*pi*1/2}"/>
         </visual>
@@ -184,9 +206,9 @@
     <link name="${prefix}_upper_leg_link">
         <visual>
-            <xacro:default_geometry cad_file="FP04-F4"/>
+            <default_geometry cad_file="FP04-F4"/>
             <origin xyz="0 0 0" rpy="${-1*reflect*pi/2} ${-1*reflect*pi/2} ${-pi/2}"/>
         </visual>
         <visual>
-            <xacro:default_geometry cad_file="FP04-F1"/>
+            <default_geometry cad_file="FP04-F1"/>
             <origin xyz="${reflect*0.075} 0.0145 0" rpy="${pi/2} ${reflect*pi/2} ${-1*reflect*pi/2}"/>
         </visual>
@@ -214,13 +236,13 @@
         <!-- Motor 13[r] 14[l] -->
         <visual>
-            <xacro:default_geometry cad_file="AX-12"/>
+            <default_geometry cad_file="AX-12"/>
             <origin xyz="0 0 0" rpy="0 0 0"/>
         </visual>
         <visual>
-            <xacro:default_geometry cad_file="FP04-F3"/>
+            <default_geometry cad_file="FP04-F3"/>
             <origin xyz="${reflect*0.019} -0.0145 0" rpy="0 0 ${reflect*pi/2}"/>
         </visual>
         <visual>
-            <xacro:default_geometry cad_file="FP04-F4"/>
+            <default_geometry cad_file="FP04-F4"/>
             <origin xyz="${reflect*0.071} -0.0145 0" rpy="${reflect*pi/2} ${reflect*pi/2} ${-pi/2}"/>
         </visual>
@@ -248,22 +270,22 @@
         <!-- Motor 15[r] 16[l] -->
         <visual>
-            <xacro:default_geometry cad_file="AX-12"/>
+            <default_geometry cad_file="AX-12"/>
             <origin xyz="0 0 0" rpy=" ${(reflect-1)*pi*-1/2}  ${(reflect+1)*pi*1/2} ${-pi/2}"/>
         </visual>
         <visual>
-            <xacro:default_geometry cad_file="FP04-F7"/>
+            <default_geometry cad_file="FP04-F7"/>
             <origin xyz="${-1*reflect*0.0145} 0.019 0" rpy="${pi} ${(reflect-1)*pi*-1/2} 0"/>
         </visual>
         <!-- Motor 17[r] 18[l] -->
         <visual>
-            <xacro:default_geometry cad_file="AX-12"/>
+            <default_geometry cad_file="AX-12"/>
             <origin xyz="0 -0.032 0" rpy="0 ${reflect*pi/2} ${-1*reflect*pi/2}"/>
         </visual>
         <visual>
-            <xacro:default_geometry cad_file="FP04-F6"/>
+            <default_geometry cad_file="FP04-F6"/>
             <origin xyz="${-1*reflect*0.0145} -0.048 ${reflect*0.019}" rpy="${-1*reflect*pi/2} 0 ${-pi/2}"/>
         </visual>
         <visual>
-            <xacro:default_geometry cad_file="FP04-F6"/>
+            <default_geometry cad_file="FP04-F6"/>
             <origin xyz="${-1*reflect*0.0145} -0.048 ${-1*reflect*0.019}" rpy="${reflect*pi/2} 0 ${-pi/2}"/>
         </visual>
@@ -284,9 +306,9 @@
     <link name="${prefix}_ankle_lateral_link">
         <visual>
-            <xacro:default_geometry cad_file="BPF-BU"/>
+            <default_geometry cad_file="BPF-BU"/>
             <origin xyz="0 0 0.015" rpy="${pi/2} 0 0"/>
         </visual>
         <visual>
-            <xacro:default_geometry cad_file="FP04-F5"/>
+            <default_geometry cad_file="FP04-F5"/>
             <origin xyz="0 0 -0.0155" rpy="${-1*reflect*pi/2} ${(reflect-1)*pi*-1/2}  ${-pi/2}"/>
         </visual>
@@ -316,5 +338,5 @@
     <link name="r_shoulder_swing_link">
         <visual>
-            <xacro:default_geometry cad_file="FP04-F1"/>
+            <default_geometry cad_file="FP04-F1"/>
             <origin xyz="0 0.014 0.044" rpy="0 ${pi} ${pi}"/>
         </visual>
@@ -335,5 +357,5 @@
     <link name="l_shoulder_swing_link">
         <visual>
-            <xacro:default_geometry cad_file="FP04-F1"/>
+            <default_geometry cad_file="FP04-F1"/>
             <origin xyz="0 0.014 0.044" rpy="0 ${pi} ${pi}"/>
         </visual>
@@ -354,21 +376,21 @@
     <link name="r_upper_arm_link">
         <visual>
-            <xacro:default_geometry cad_file="AX-12"/>
+            <default_geometry cad_file="AX-12"/>
             <origin xyz="0 0 0" rpy="0 0 ${pi/2}"/>
         </visual>
         <visual>
-            <xacro:default_geometry cad_file="BPF-BU"/>
+            <default_geometry cad_file="BPF-BU"/>
             <origin xyz="0 0 -0.0185" rpy="${-pi/2} 0 ${pi/2}"/>
         </visual>
         <visual>
-            <xacro:default_geometry cad_file="BPF-WA"/>
+            <default_geometry cad_file="BPF-WA"/>
             <origin xyz="0 0 -0.019" rpy="${-pi/2} 0 ${pi/2}"/>
         </visual>
         <visual>
-            <xacro:default_geometry cad_file="FP04-F3"/>
+            <default_geometry cad_file="FP04-F3"/>
             <origin xyz="0.0415 0 0" rpy="0 0 ${pi/2}"/>
         </visual>
         <visual>
-            <xacro:default_geometry cad_file="FP04-F2"/>
+            <default_geometry cad_file="FP04-F2"/>
             <origin xyz="0.0675 0 0" rpy="${-pi/2} ${pi/2} ${pi/2}"/>
         </visual>
@@ -395,21 +417,21 @@
     <link name="l_upper_arm_link">
         <visual>
-            <xacro:default_geometry cad_file="AX-12"/>
+            <default_geometry cad_file="AX-12"/>
             <origin xyz="0 0 0" rpy="${pi} 0 ${-pi/2}"/>
         </visual>
         <visual>
-            <xacro:default_geometry cad_file="BPF-BU"/>
+            <default_geometry cad_file="BPF-BU"/>
             <origin xyz="0 0 0.0185" rpy="${pi/2} 0 ${pi/2}"/>
         </visual>
         <visual>
-            <xacro:default_geometry cad_file="BPF-WA"/>
+            <default_geometry cad_file="BPF-WA"/>
             <origin xyz="0 0 0.019" rpy="${pi/2} 0 ${pi/2}"/>
         </visual>
         <visual>
-            <xacro:default_geometry cad_file="FP04-F3"/>
+            <default_geometry cad_file="FP04-F3"/>
             <origin xyz="0.0415 0 0" rpy="${pi} 0 ${-pi/2}"/>
         </visual>
         <visual>
-            <xacro:default_geometry cad_file="FP04-F2"/>
+            <default_geometry cad_file="FP04-F2"/>
             <origin xyz="0.0675 0 0" rpy="${pi/2} ${pi/2} ${-pi/2}"/>
         </visual>
@@ -437,17 +459,17 @@
         <!-- Motor 5 -->
         <visual>
-            <xacro:default_geometry cad_file="AX-12"/>
+            <default_geometry cad_file="AX-12"/>
             <origin xyz="0 0 0" rpy="0 0 ${pi/2}"/>
         </visual>
         <visual>
-            <xacro:default_geometry cad_file="BPF-BU"/>
+            <default_geometry cad_file="BPF-BU"/>
             <origin xyz="0 0 -0.0185" rpy="${-pi/2} 0 ${pi/2}"/>
         </visual>
         <visual>
-            <xacro:default_geometry cad_file="BPF-WA"/>
+            <default_geometry cad_file="BPF-WA"/>
             <origin xyz="0 0 -0.019" rpy="${-pi/2} 0 ${pi/2}"/>
         </visual>
         <visual>
-            <xacro:default_geometry cad_file="FP04-F3"/>
+            <default_geometry cad_file="FP04-F3"/>
             <origin xyz="0.0415 0 0" rpy="0 0 ${pi/2}"/>
         </visual>
@@ -469,17 +491,17 @@
         <!-- Motor 6 -->
         <visual>
-            <xacro:default_geometry cad_file="AX-12"/>
+            <default_geometry cad_file="AX-12"/>
             <origin xyz="0 0 0" rpy="${pi} 0 ${-pi/2}"/>
         </visual>
         <visual>
-            <xacro:default_geometry cad_file="BPF-BU"/>
+            <default_geometry cad_file="BPF-BU"/>
             <origin xyz="0 0 0.0185" rpy="${pi/2} 0 ${pi/2}"/>
         </visual>
         <visual>
-            <xacro:default_geometry cad_file="BPF-WA"/>
+            <default_geometry cad_file="BPF-WA"/>
             <origin xyz="0 0 0.019" rpy="${pi/2} 0 ${pi/2}"/>
         </visual>
         <visual>
-            <xacro:default_geometry cad_file="FP04-F3"/>
+            <default_geometry cad_file="FP04-F3"/>
             <origin xyz="0.0415 0 0" rpy="${pi} 0 ${-pi/2}"/>
         </visual>
@@ -500,5 +522,5 @@
     <link name="r_hand_link">
         <visual>
-            <xacro:default_geometry cad_file="FP04-F11"/>
+            <default_geometry cad_file="FP04-F11"/>
             <origin xyz="0.0415 0 0" rpy="${pi} ${-pi/2} 0"/>
         </visual>
@@ -525,5 +547,5 @@
     <link name="l_hand_link">
         <visual>
-            <xacro:default_geometry cad_file="FP04-F11"/>
+            <default_geometry cad_file="FP04-F11"/>
             <origin xyz="0.0415 0 0" rpy="0 ${-pi/2} ${pi}"/>
         </visual>
