Commit message: Add inertia retrieved from SolidWorks app.
 - Files (xml) in inertia directory are generated automatically
 (do not change by hands).

File: std_parts.xacro (robot description, xacro)
@@ -2,4 +2,7 @@
 <!-- Standard Bioloid parts -->
 <robot xmlns:xacro="http://www.ros.org/wiki/xacro">
+	<!-- Import mass property (inertia) -->
+	<xacro:include filename="$(find bioloid_typea_description)/inertia/Torso.xacro"/>
+	<xacro:include filename="$(find bioloid_typea_description)/inertia/F12.xacro"/>
     <!-- Torso -->
     <link name="torso_link">
@@ -75,4 +78,6 @@
             </geometry>
         </collision>
+        <xacro:torso_inertial/>
+        <!--
         <inertial>
             <origin xyz="-0.003053 -0.038651 -0.019268" />
@@ -80,4 +85,5 @@
             <inertia ixx="3.1081800"  ixy="-0.25460189"  ixz="2.0318174" iyy="6.3787776" iyz="0.16417863" izz="5.3316425" />
         </inertial>
+        -->
     </link>
     <!-- Right foot -->
@@ -93,4 +99,6 @@
             </geometry>
         </collision>
+        <xacro:foot_right_inertial/>
+        <!--
         <inertial>
             <origin xyz="-0.025995 -0.009506 -0.000503" />
@@ -98,4 +106,5 @@
             <inertia ixx="0.12079175"  ixy="-0.00079781067"  ixz="-0.00039322246" iyx="-0.00079781067" iyy="0.10885465" iyz="0.0070770117" izx="-0.00039322246" izy="0.0070770117" izz="0.041871103" />
         </inertial>
+        -->
     </link>
     <!-- Left foot -->
@@ -111,4 +120,6 @@
             </geometry>
         </collision>
+        <xacro:foot_left_inertial/>
+        <!--
         <inertial>
             <origin xyz="-0.025995 -0.009506 -0.000503" />
@@ -116,4 +127,5 @@
             <inertia ixx="0.12079175"  ixy="-0.00079781067"  ixz="-0.00039322246" iyx="-0.00079781067" iyy="0.10885465" iyz="0.0070770117" izx="-0.00039322246" izy="0.0070770117" izz="0.041871103" />
         </inertial>
+        -->
     </link>
 </robot>

File: typea.urdf (robot description, URDF)
Before this commit: robot typea, 25 links, 24 joints
Links:
- link l_ankle_lateral_link: mass 0.0794462 -> 0.0373560220
- link l_ankle_swing_link: mass 0.16710792 -> 0.1370485873
- link l_foot_link: mass 0.0794462 -> 0.0373560220
- link l_hand_link: mass 0.010 -> 0.0060600633
- link l_hip_lateral_link: mass 0.11904336 -> 0.1370485873
- link l_hip_twist_link: mass 0.167 -> 0.0151038725
- link l_lower_arm_link: mass 0.059288504 -> 0.0764574147
- link l_lower_leg_link: mass 0.070309794 -> 0.0865217867
- link l_shoulder_swing_link: mass 0.025913024 -> 0.0119189163
- link l_upper_arm_link: mass 0.16837715 -> 0.0764574147
- link l_upper_leg_link: mass 0.11904336 -> 0.0311530844
- link r_ankle_lateral_link: mass 0.0794462 -> 0.0373560220
- link r_ankle_swing_link: mass 0.16710792 -> 0.1370485873
- link r_foot_link: mass 0.0794462 -> 0.0373560220
- link r_hand_link: mass 0.010 -> 0.0060600633
- link r_hip_lateral_link: mass 0.11904336 -> 0.1370485873
- link r_hip_twist_link: mass 0.167 -> 0.0151038725
- link r_lower_arm_link: mass 0.059288504 -> 0.0706166158
- link r_lower_leg_link: mass 0.070309794 -> 0.0865217867
- link r_shoulder_swing_link: mass 0.025913024 -> 0.0119189163
- link r_upper_arm_link: mass 0.16837715 -> 0.0764574147
- link r_upper_leg_link: mass 0.11904336 -> 0.0311530844
- link torso_link: mass 0.97559947 -> 0.6954053293
Joints:
- joint l_ankle_lateral_joint: origin xyz=0 0 0 rpy=-1.570795 0 0 -> xyz=0 0 0 rpy=-1.57079632679 0 0
- joint l_ankle_swing_joint: origin xyz=-0.071 -0.0145 0 rpy=3.14159 0 0 -> xyz=-0.071 -0.0145 0 rpy=3.14159265359 0 0
- joint l_hip_lateral_joint: origin xyz=0 0 0.05 rpy=1.570795 0 0 -> xyz=0 0 0.05 rpy=1.57079632679 0 0
- joint l_hip_swing_joint: origin xyz=0 0 0 rpy=1.570795 0 -1.570795 -> xyz=0 0 0 rpy=1.57079632679 0 -1.57079632679
- joint l_hip_twist_joint: origin xyz=0 0.0385 -0.0655 rpy=0 3.14159 -1.570795 -> xyz=0 0.0385 -0.0655 rpy=0 3.14159265359 -1.57079632679
- joint l_shoulder_lateral_joint: origin xyz=0 0.014 0.044 rpy=0 -1.570795 0 -> xyz=0 0.014 0.044 rpy=0 -1.57079632679 0
- joint l_shoulder_swing_joint: limit lower=-1 upper=1.570795 effort=2.8 velocity=1.0 -> lower=-1 upper=1.57079632679 effort=2.8 velocity=1.0; origin xyz=0 0.032 0 rpy=-1.570795 -1.570795 0 -> xyz=0 0.032 0 rpy=-1.57079632679 -1.57079632679 0
- joint r_ankle_lateral_joint: origin xyz=0 0 0 rpy=-1.570795 0 0 -> xyz=0 0 0 rpy=-1.57079632679 0 0
- joint r_ankle_swing_joint: origin xyz=0.071 -0.0145 0 rpy=3.14159 0 0 -> xyz=0.071 -0.0145 0 rpy=3.14159265359 0 0
- joint r_hip_lateral_joint: origin xyz=0 0 0.05 rpy=-1.570795 0 0 -> xyz=0 0 0.05 rpy=-1.57079632679 0 0
- joint r_hip_swing_joint: origin xyz=0 0 0 rpy=1.570795 0 -1.570795 -> xyz=0 0 0 rpy=1.57079632679 0 -1.57079632679
- joint r_hip_twist_joint: origin xyz=0 -0.0385 -0.0655 rpy=0 3.14159 1.570795 -> xyz=0 -0.0385 -0.0655 rpy=0 3.14159265359 1.57079632679
- joint r_shoulder_lateral_joint: origin xyz=0 0.014 0.044 rpy=0 -1.570795 0 -> xyz=0 0.014 0.044 rpy=0 -1.57079632679 0
- joint r_shoulder_swing_joint: limit lower=-1 upper=1.570795 effort=2.8 velocity=1.0 -> lower=-1 upper=1.57079632679 effort=2.8 velocity=1.0; origin xyz=0 -0.032 0 rpy=1.570795 1.570795 0 -> xyz=0 -0.032 0 rpy=1.57079632679 1.57079632679 0

File: typea.xacro (robot description, xacro)
@@ -1,7 +1,23 @@
 <?xml version="1.0"?>
 <robot xmlns:xacro="http://www.ros.org/wiki/xacro" name="typea">
+	<!-- Import mass property (inertia) -->
+	<xacro:include filename="$(find bioloid_typea_description)/inertia/Torso.xacro"/>
+	<xacro:include filename="$(find bioloid_typea_description)/inertia/F1.xacro"/>
+	<xacro:include filename="$(find bioloid_typea_description)/inertia/F5.xacro"/>
+	<xacro:include filename="$(find bioloid_typea_description)/inertia/F12.xacro"/>
+	<xacro:include filename="$(find bioloid_typea_description)/inertia/F11.xacro"/>
+	<xacro:include filename="$(find bioloid_typea_description)/inertia/upperarm.xacro"/>
+	<xacro:include filename="$(find bioloid_typea_description)/inertia/upperleg.xacro"/>
+	<xacro:include filename="$(find bioloid_typea_description)/inertia/L_Foot.xacro"/>
+	<xacro:include filename="$(find bioloid_typea_description)/inertia/R_Foot.xacro"/>
+	<xacro:include filename="$(find bioloid_typea_description)/inertia/L_lowerarm.xacro"/>
+	<xacro:include filename="$(find bioloid_typea_description)/inertia/R_lowerarm.xacro"/>
+	<xacro:include filename="$(find bioloid_typea_description)/inertia/L_Tibia.xacro"/>
+	<xacro:include filename="$(find bioloid_typea_description)/inertia/R_Tibia.xacro"/>
+	<xacro:include filename="$(find bioloid_typea_description)/inertia/L_hip-R_ankle.xacro"/>
+	<xacro:include filename="$(find bioloid_typea_description)/inertia/R_hip-L_ankle.xacro"/>
     <!-- Import gazebo_ros_control plugin -->
     <xacro:include filename="$(find bioloid_typea_description)/gazebo.xacro" ns="gazebo"/>
-    <xacro:property name="pi" value="3.14159"/>
+    <!--  <xacro:property name="pi" value="3.14159"/> -->
     <xacro:property name="cad_dir" value="file://$(find bioloid_typea_description)/assets/cad"/>
     <!-- Typically, STL/DAE model units are in mm, but RViz units are in m, hence models must be scaled down by 1000. -->
@@ -143,5 +159,5 @@
     </xacro:macro>
     <!-- Links MACRO -->
-    <xacro:macro name="hip_lateral_link" params="prefix reflect x_offset y_offset z_offset">
+    <xacro:macro name="hip_lateral_link" params="prefix reflect x_offset y_offset z_offset *inertial">
     <link name="${prefix}_hip_lateral_link">
         <!-- Motor 9[r] 10[l] -->
@@ -177,4 +193,6 @@
             </geometry>
         </collision>
+        <xacro:insert_block name="inertial" />
+        <!--
         <inertial>
             <origin xyz="0.000079 0.018242 0.013873" />
@@ -182,4 +200,5 @@
             <inertia ixx="0.097950272"  ixy="0.0012119368"  ixz="-0.00021223016" iyx="0.00122119368" iyy="0.032848287" iyz="-0.0019474021" izx="-0.00021223016" izy="-0.0019474021" izz="0.11493509" />
         </inertial>
+        -->
     </link>
     </xacro:macro>
@@ -196,4 +215,6 @@
             </geometry>
         </collision>
+        <xacro:hip_twist_inertial/>
+        <!--
         <inertial>
             <origin xyz="0.000000 0.000480 0.018437" />
@@ -201,4 +222,5 @@
             <inertia ixx="0.12259691"  ixy="0.00071127469"  ixz="0.00081143913" iyx="0.00071127469" iyy="0.11066637" iyz="-0.0071635476" izx="0.00081143913" izy="-0.0071635476" izz="0.041877668" />
         </inertial>
+        -->
     </link>
     </xacro:macro>
@@ -225,4 +247,6 @@
             </geometry>
         </collision>
+        <xacro:upperleg_inertial/>
+        <!--
         <inertial>
             <origin xyz="-0.062965 -0.000323 0.000692" />
@@ -230,7 +254,8 @@
             <inertia ixx="0.097950272"  ixy="0.0012119368"  ixz="-0.00021223016" iyx="0.00122119368" iyy="0.032848287" iyz="-0.0019474021" izx="-0.00021223016" izy="-0.0019474021" izz="0.11493509" />
         </inertial>
-    </link>
-    </xacro:macro>
-    <xacro:macro name="lower_leg_link" params="prefix reflect x_offset y_offset z_offset">
+        -->
+    </link>
+    </xacro:macro>
+    <xacro:macro name="lower_leg_link" params="prefix reflect x_offset y_offset z_offset *inertial">
     <link name="${prefix}_lower_leg_link">
         <!-- Motor 13[r] 14[l] -->
@@ -259,4 +284,6 @@
             </geometry>
         </collision>
+        <xacro:insert_block name="inertial" />
+        <!--
         <inertial>
             <origin xyz="-0.053955 0.006548 -0.000592" />
@@ -264,7 +291,8 @@
             <inertia ixx="0.093369608"  ixy="-0.00093567395"  ixz="-0.00023992085" iyx="-0.00093567395" iyy="0.046295534" iyz="-0.012858493" izx="-0.00023992085" izy="-0.012858493" izz="0.11351516" />
         </inertial>
-    </link>
-    </xacro:macro>
-    <xacro:macro name="ankle_swing_link" params="prefix reflect x_offset y_offset z_offset">
+        -->
+    </link>
+    </xacro:macro>
+    <xacro:macro name="ankle_swing_link" params="prefix reflect x_offset y_offset z_offset *inertial">
     <link name="${prefix}_ankle_swing_link">
         <!-- Motor 15[r] 16[l] -->
@@ -296,4 +324,6 @@
             </geometry>
         </collision>
+        <xacro:insert_block name="inertial" />
+        <!--
         <inertial>
             <origin xyz="-0.000214 -0.018536 0.013873" />
@@ -301,7 +331,8 @@
             <inertia ixx="0.12079175"  ixy="-0.00079781067"  ixz="-0.00039322246" iyx="-0.00079781067" iyy="0.10885465" iyz="0.0070770117" izx="-0.00039322246" izy="0.0070770117" izz="0.041871103" />
         </inertial>
-    </link>
-    </xacro:macro>
-    <xacro:macro name="ankle_lateral_link" params="prefix reflect x_offset y_offset z_offset">
+        -->
+    </link>
+    </xacro:macro>
+    <xacro:macro name="ankle_lateral_link" params="prefix reflect x_offset y_offset z_offset *inertial">
     <link name="${prefix}_ankle_lateral_link">
         <visual>
@@ -319,4 +350,6 @@
             </geometry>
         </collision>
+        <xacro:insert_block name="inertial" />
+        <!--
         <inertial>
             <origin xyz="-0.025995 -0.009506 -0.000503" />
@@ -324,4 +357,5 @@
             <inertia ixx="0.12079175"  ixy="-0.00079781067"  ixz="-0.00039322246" iyx="-0.00079781067" iyy="0.10885465" iyz="0.0070770117" izx="-0.00039322246" izy="0.0070770117" izz="0.041871103" />
         </inertial>
+        -->
     </link>
     </xacro:macro>
@@ -347,4 +381,6 @@
             </geometry>
         </collision>
+        <xacro:shoulder_right_inertial/>
+        <!--
         <inertial>
             <origin xyz="-0.013522619 0.010264050 0.0013935747"/>
@@ -352,4 +388,5 @@
             <inertia  ixx="0.0097758165" ixy="0.0016911839"  ixz="-0.0016911839"  iyy="0.010511104"  iyz="0.00033406955"  izz="0.005476798"/>
         </inertial>
+        -->
     </link>
     <!-- Torso to left shoulder -->
@@ -366,4 +403,6 @@
             </geometry>
         </collision>
+        <xacro:shoulder_left_inertial/>
+        <!--
         <inertial>
             <origin xyz="-0.013522619 0.010264050 0.0013935747"/>
@@ -371,4 +410,5 @@
             <inertia  ixx="0.0097758165" ixy="0.0016911839"  ixz="-0.0016911839"  iyy="0.010511104"  iyz="0.00033406955"  izz="0.005476798"/>
         </inertial>
+        -->
     </link>
     <!-- Right shoulder to upper arm -->
@@ -407,9 +447,12 @@
             </geometry>
         </collision>
-        <inertial>
-      <origin xyz="-0.036239 0.000734 -0.000660" />
-      <mass value="0.16837715"/>
-      <inertia ixx="0.12202839"  ixy="-0.0020812626"  ixz="-0.00088143449" iyx="-0.0020812626" iyy="0.038088441" iyz="0.0018251448" izx="-0.00088143449" izy="0.0018251448" izz="0.11340830" />
-        </inertial>
+        <xacro:upperarm_right_inertial/>
+        <!--
+        <inertial>
+      	<origin xyz="-0.036239 0.000734 -0.000660" />
+      	<mass value="0.16837715"/>
+      	<inertia ixx="0.12202839"  ixy="-0.0020812626"  ixz="-0.00088143449" iyx="-0.0020812626" iyy="0.038088441" iyz="0.0018251448" izx="-0.00088143449" izy="0.0018251448" izz="0.11340830" />
+        </inertial>
+        -->
     </link>
     <!-- Left shoulder to upper arm -->
@@ -448,9 +491,12 @@
             </geometry>
         </collision>
-        <inertial>
-      <origin xyz="-0.036239 0.000734 -0.000660" />
-      <mass value="0.16837715"/>
-      <inertia ixx="0.12202839"  ixy="-0.0020812626"  ixz="-0.00088143449" iyx="-0.0020812626" iyy="0.038088441" iyz="0.0018251448" izx="-0.00088143449" izy="0.0018251448" izz="0.11340830" />
-        </inertial>
+        <xacro:upperarm_left_inertial/>
+        <!--
+        <inertial>
+      	<origin xyz="-0.036239 0.000734 -0.000660" />
+      	<mass value="0.16837715"/>
+      	<inertia ixx="0.12202839"  ixy="-0.0020812626"  ixz="-0.00088143449" iyx="-0.0020812626" iyy="0.038088441" iyz="0.0018251448" izx="-0.00088143449" izy="0.0018251448" izz="0.11340830" />
+        </inertial>
+        -->
     </link>
     <!-- Right upper arm to lower arm -->
@@ -480,4 +526,6 @@
             </geometry>
         </collision>
+        <xacro:lowerarm_right_inertial/>
+        <!--
         <inertial>
             <origin xyz="0.000000 0.000000 0.000000" />
@@ -485,4 +533,5 @@
             <inertia ixx="0.086855267"  ixy="0.0053020311"  ixz="0.00043636051" iyx="0.0053020311" iyy="0.021192085" iyz="-0.0064855932" izx="0.00043636051" izy="-0.0064855932" izz="0.086845450" />
         </inertial>
+        -->
     </link>
     <!-- Left upper arm to lower arm -->
@@ -512,4 +561,6 @@
             </geometry>
         </collision>
+        <xacro:upperarm_left_inertial/>
+        <!--
         <inertial>
             <origin xyz="0.000000 0.000000 0.000000" />
@@ -517,4 +568,5 @@
             <inertia ixx="0.086855267"  ixy="0.0053020311"  ixz="0.00043636051" iyx="0.0053020311" iyy="0.021192085" iyz="-0.0064855932" izx="0.00043636051" izy="-0.0064855932" izz="0.086845450" />
         </inertial>
+        -->
     </link>
     <!-- Right lower arm to hand -->
@@ -537,4 +589,6 @@
             </geometry>
         </collision>
+        <xacro:arm_right_inertial/>
+        <!--
         <inertial>
             <origin xyz="0.045838 -0.013490 0.006666"/>
@@ -542,4 +596,5 @@
             <inertia ixx="0.12202839"  ixy="-0.0020812626"  ixz="-0.00088143449" iyx="-0.0020812626" iyy="0.038088441" iyz="0.0018251448" izx="-0.00088143449" izy="0.0018251448" izz="0.11340830" />
         </inertial>
+        -->
     </link>
     <!-- Left lower arm to hand -->
@@ -562,4 +617,6 @@
             </geometry>
         </collision>
+        <xacro:arm_left_inertial/>
+        <!--
         <inertial>
             <origin xyz="0.045838 -0.013490 0.006666"/>
@@ -567,4 +624,5 @@
             <inertia ixx="0.12202839"  ixy="-0.0020812626"  ixz="-0.00088143449" iyx="-0.0020812626" iyy="0.038088441" iyz="0.0018251448" izx="-0.00088143449" izy="0.0018251448" izz="0.11340830" />
         </inertial>
+        -->
     </link>
     <!-- Torso to right hip twist -->
@@ -576,8 +634,12 @@
     <!-- Right hip twist to hip lateral -->
     <xacro:hip_lateral_joint prefix="r" reflect="1"/>
-    <xacro:hip_lateral_link prefix="r" reflect="1" x_offset="0" y_offset="0" z_offset="0.0353"/>
+    <xacro:hip_lateral_link prefix="r" reflect="1" x_offset="0" y_offset="0" z_offset="0.0353">
+    	<xacro:hip_right_inertial/>
+    </xacro:hip_lateral_link>
     <!-- Left hip twist to hip lateral -->
     <xacro:hip_lateral_joint prefix="l" reflect="-1"/>
-    <xacro:hip_lateral_link prefix="l" reflect="-1" x_offset="0" y_offset="0" z_offset="0.0353"/>
+    <xacro:hip_lateral_link prefix="l" reflect="-1" x_offset="0" y_offset="0" z_offset="0.0353">
+		<xacro:hip_left_inertial/>
+    </xacro:hip_lateral_link>
     <!-- Right hip lateral to upper leg -->
     <xacro:hip_swing_joint prefix="r" reflect="1"/>
@@ -588,20 +650,32 @@
     <!-- Right upper leg to lower leg -->
     <xacro:knee_joint prefix="r" reflect="1"/>
-    <xacro:lower_leg_link prefix="r" reflect="1" x_offset="0" y_offset="0" z_offset="0"/>
+    <xacro:lower_leg_link prefix="r" reflect="1" x_offset="0" y_offset="0" z_offset="0">
+    	<xacro:tibia_right_inertial/>
+    </xacro:lower_leg_link>
     <!-- Left upper leg to lower leg -->
     <xacro:knee_joint prefix="l" reflect="-1"/>
-    <xacro:lower_leg_link prefix="l" reflect="-1" x_offset="0" y_offset="0" z_offset="0"/>
+    <xacro:lower_leg_link prefix="l" reflect="-1" x_offset="0" y_offset="0" z_offset="0">
+    	<xacro:tibia_left_inertial/>
+    </xacro:lower_leg_link>
     <!-- Right lower leg to ankle swing -->
     <xacro:ankle_swing_joint prefix="r" reflect="1"/>
-    <xacro:ankle_swing_link prefix="r" reflect="1" x_offset="0" y_offset="0" z_offset="0"/>
+    <xacro:ankle_swing_link prefix="r" reflect="1" x_offset="0" y_offset="0" z_offset="0">
+    	<xacro:ankle_right_inertial/>
+    </xacro:ankle_swing_link>
     <!-- Left lower leg to ankle swing -->
     <xacro:ankle_swing_joint prefix="l" reflect="-1"/>
-    <xacro:ankle_swing_link prefix="l" reflect="-1" x_offset="0" y_offset="0" z_offset="0"/>
+    <xacro:ankle_swing_link prefix="l" reflect="-1" x_offset="0" y_offset="0" z_offset="0">
+    	<xacro:ankle_left_inertial/>
+    </xacro:ankle_swing_link>
     <!-- Right ankle swing to ankle lateral -->
     <xacro:ankle_lateral_joint prefix="r" reflect="1"/>
-    <xacro:ankle_lateral_link prefix="r" reflect="1" x_offset="0" y_offset="0" z_offset="0"/>
+    <xacro:ankle_lateral_link prefix="r" reflect="1" x_offset="0" y_offset="0" z_offset="0">
+    	<xacro:foot_right_inertial/>
+    </xacro:ankle_lateral_link>
     <!-- Left ankle swing to ankle lateral -->
     <xacro:ankle_lateral_joint prefix="l" reflect="-1"/>
-    <xacro:ankle_lateral_link prefix="l" reflect="-1" x_offset="0" y_offset="0" z_offset="0"/>
+    <xacro:ankle_lateral_link prefix="l" reflect="-1" x_offset="0" y_offset="0" z_offset="0">
+    	<xacro:foot_left_inertial/>
+    </xacro:ankle_lateral_link>
     <!-- Right ankle lateral to foot -->
     <xacro:foot_joint prefix="r"/>
