Commit message: Move Imu has a child under base_link.
 - This matches better ROS standard:
  earth -> map -> odom -> base_link

File: gazebo.xacro (robot description, xacro)
@@ -10,8 +10,9 @@
 		    <alwaysOn>true</alwaysOn>
 		    <bodyName>imu_link</bodyName>
-		    <topicName>imu</topicName>
+		    <topicName>/typea/imu</topicName>
 		    <serviceName>imu_service</serviceName>
 		    <gaussianNoise>0.0</gaussianNoise>
 		    <updateRate>20.0</updateRate>
+		    <visualize>true</visualize>
 		</plugin>
     </gazebo>

File: typea.urdf (robot description, URDF)
Before this commit: robot typea, 25 links, 24 joints
Links:
- link imu_link: mass None -> 0.001; geometry collision box size=.01 .01 .01; visual box size=0.04 0.02 0.005
Joints:
- joint imu_to_base_joint: axis (none) -> 1 0 0; child base_link -> imu_link; origin xyz=0.01 0 0.0788 rpy=0 0 0 -> xyz=0 0 0.05 rpy=0 0 0; parent imu_link -> base_link

File: typea.xacro (robot description, xacro)
@@ -36,10 +36,12 @@
     <!-- IMU -->
     <joint name="imu_to_base_joint" type="fixed">
-        <parent link="imu_link"/>
-        <origin xyz="0.01 0 0.0788" rpy="0 0 0"/>
-        <child link="base_link"/>
+        <axis xyz="1 0 0"/>
+        <origin xyz="0 0 0.05" rpy="0 0 0"/>
+        <parent link="base_link"/>
+        <child link="imu_link"/>
     </joint>
     <link name="imu_link">
         <visual>
+            <origin rpy="0 0 0" xyz="0 0 0"/>
             <geometry>
                 <box size="0.04 0.02 0.005"/>
@@ -49,9 +51,15 @@
             </material>
         </visual>
-        <!--<inertial>
-            <origin xyz="0 0 0"/>
-            <mass value="1.0"/>
-            <inertia  ixx="0.001" ixy="0.0"  ixz="0.0"  iyy="0.001"  iyz="0.0"  izz="0.001"/>
-        </inertial>-->
+          <collision>
+	    <origin rpy="0 0 0" xyz="0 0 0"/>
+	        <geometry>
+	        <box size=".01 .01 .01"/>
+	        </geometry>
+	    </collision>
+	  <inertial>
+	    <mass value="0.001"/>
+	    <origin rpy="0 0 0" xyz="0 0 0"/>
+	    <inertia ixx="0.0001" ixy="0" ixz="0" iyy="0.000001" iyz="0" izz="0.0001"/>
+	  </inertial>
     </link>
     <xacro:macro name="shoulder_swing_joint" params="prefix reflect">
