Commit message: Fix limit for knee actuators.
 - no need to invert rotation axes anymore.
 - now the sim and the real robot behave the same.

File: typea.urdf (robot description, URDF)
Before this commit: robot typea, 25 links, 24 joints
Joints:
- joint l_knee_joint: axis 0 0 -1 -> 0 0 1; limit lower=-0.0 upper=1.1 effort=10 velocity=5.6548668 -> lower=-2 upper=0 effort=10 velocity=5.6548668
- joint r_knee_joint: axis 0 0 -1 -> 0 0 1; limit lower=-1.1 upper=-0.0 effort=10 velocity=5.6548668 -> lower=0 upper=2 effort=10 velocity=5.6548668

File: typea.xacro (robot description, xacro)
@@ -104,7 +104,7 @@
             <parent link="${prefix}_upper_leg_link"/>
             <origin xyz="${reflect*0.075} 0.0145 0" rpy="0 0 0"/>
-            <axis xyz="0 0 -1"/>
+            <axis xyz="0 0 1"/>
             <child link="${prefix}_lower_leg_link"/>
-            <limit lower="${-0.55*(1+reflect)}" upper="${-0.55*(-1+reflect)}" effort="10" velocity="5.6548668"/>
+            <limit lower="${-1+reflect}" upper="${1+reflect}" effort="10" velocity="5.6548668"/>
         </joint>
     </xacro:macro>

Commit message: Relax limit for hip, knee, ankle

File: typea.urdf (robot description, URDF)
Before this commit: robot typea, 25 links, 24 joints
Joints:
- joint l_ankle_swing_joint: limit lower=-1.0 upper=0.4 effort=10 velocity=5.6548668 -> lower=-2.0 upper=0.4 effort=10 velocity=5.6548668
- joint l_hip_swing_joint: limit lower=-0.4 upper=1.0 effort=10 velocity=5.6548668 -> lower=-0.4 upper=2.0 effort=10 velocity=5.6548668
- joint r_ankle_swing_joint: limit lower=-0.4 upper=1.0 effort=10 velocity=5.6548668 -> lower=-0.4 upper=2.0 effort=10 velocity=5.6548668
- joint r_hip_swing_joint: limit lower=-1.0 upper=0.4 effort=10 velocity=5.6548668 -> lower=-2.0 upper=0.4 effort=10 velocity=5.6548668

File: typea.xacro (robot description, xacro)
@@ -97,5 +97,5 @@
             <xacro:z_rot/>
             <child link="${prefix}_upper_leg_link"/>
-            <limit lower="${-0.3*(reflect-1)-1}" upper="${-0.3*(reflect+1)+1}" effort="10" velocity="5.6548668"/>
+            <limit lower="${-0.8*(reflect-1)-2}" upper="${-0.8*(reflect+1)+2}" effort="10" velocity="5.6548668"/>
         </joint>
     </xacro:macro>
@@ -115,5 +115,5 @@
             <xacro:z_rot/>
             <child link="${prefix}_ankle_swing_link"/>
-            <limit lower="${0.3*(reflect+1)-1}" upper="${0.3*(reflect-1)+1}" effort="10" velocity="5.6548668"/>
+            <limit lower="${0.8*(reflect+1)-2}" upper="${0.8*(reflect-1)+2}" effort="10" velocity="5.6548668"/>
         </joint>
     </xacro:macro>

Commit message: Fix limit of the ankle.  - Issue was causing torso to rotate on the x axis during  lateral motion (CoM under feet).

File: typea.urdf (robot description, URDF)
Before this commit: robot typea, 25 links, 24 joints
Joints:
- joint l_ankle_lateral_joint: limit lower=-0.5 upper=0.5 effort=10 velocity=5.6548668 -> lower=-0.8 upper=0.8 effort=10 velocity=5.6548668
- joint l_hip_lateral_joint: limit lower=-0.6 upper=0.6 effort=10 velocity=5.6548668 -> lower=-0.8 upper=0.8 effort=10 velocity=5.6548668
- joint r_ankle_lateral_joint: limit lower=-0.5 upper=0.5 effort=10 velocity=5.6548668 -> lower=-0.8 upper=0.8 effort=10 velocity=5.6548668
- joint r_hip_lateral_joint: limit lower=-0.6 upper=0.6 effort=10 velocity=5.6548668 -> lower=-0.8 upper=0.8 effort=10 velocity=5.6548668

File: typea.xacro (robot description, xacro)
@@ -112,5 +112,5 @@
             <xacro:z_rot/>
             <child link="${prefix}_hip_lateral_link"/>
-            <limit lower="-0.6" upper="0.6" effort="10" velocity="5.6548668"/>
+            <limit lower="-0.8" upper="0.8" effort="10" velocity="5.6548668"/>
         </joint>
     </xacro:macro>
@@ -148,5 +148,5 @@
             <xacro:z_rot/>
             <child link="${prefix}_ankle_lateral_link"/>
-            <limit lower="-0.5" upper="0.5" effort="10" velocity="5.6548668"/>
+            <limit lower="-0.8" upper="0.8" effort="10" velocity="5.6548668"/>
         </joint>
     </xacro:macro>
