Commit message: Add files via upload

File: inertia/F1.xacro (robot description, xacro)
@@ -4,9 +4,9 @@
 <xacro:macro name="shoulder_left_inertial">
 	<inertial>
-		<mass value="0.0595945816"/>
+		<mass value="0.0119189163"/>
 		<origin xyz="-0.0109359544 -0.0123630374 0.0000000007" />
-		<inertia ixx="0.0069903407" ixy="0.0020812370" ixz="-0.0000000001"
-				iyy="0.0067210939" iyz="-0.0000000002"
-				izz="0.0054521983"/>
+		<inertia ixx="0.0699034069" ixy="0.0208123701" ixz="-0.0000000013"
+				iyy="0.0672109386" iyz="-0.0000000015"
+				izz="0.0545219826"/>
 	</inertial>
 </xacro:macro>
@@ -14,9 +14,9 @@
 <xacro:macro name="shoulder_right_inertial">
 	<inertial>
-		<mass value="0.0595945816"/>
+		<mass value="0.0119189163"/>
 		<origin xyz="-0.0109359544 0.0123630374 -0.0000000007" />
-		<inertia ixx="0.0069903407" ixy="-0.0020812370" ixz="0.0000000001"
-				iyy="0.0067210939" iyz="-0.0000000002"
-				izz="0.0054521983"/>
+		<inertia ixx="0.0699034069" ixy="-0.0208123701" ixz="0.0000000013"
+				iyy="0.0672109386" iyz="-0.0000000015"
+				izz="0.0545219826"/>
 	</inertial>
 </xacro:macro>

File: inertia/F11.xacro (robot description, xacro)
@@ -4,9 +4,9 @@
 <xacro:macro name="arm_right_inertial">
 	<inertial>
-		<mass value="0.0303003163"/>
+		<mass value="0.0060600633"/>
 		<origin xyz="-0.0070414665 -0.0217364083 -0.0000000095" />
-		<inertia ixx="0.0054448143" ixy="0.0011266691" ixz="0.0000000017"
-				iyy="0.0013220979" iyz="-0.0000000025"
-				izz="0.0053756998"/>
+		<inertia ixx="0.0544481426" ixy="0.0112666910" ixz="0.0000000167"
+				iyy="0.0132209786" iyz="-0.0000000248"
+				izz="0.0537569983"/>
 	</inertial>
 </xacro:macro>
@@ -14,9 +14,9 @@
 <xacro:macro name="arm_left_inertial">
 	<inertial>
-		<mass value="0.0303003163"/>
+		<mass value="0.0060600633"/>
 		<origin xyz="-0.0070414665 0.0217364083 0.0000000095" />
-		<inertia ixx="0.0054448143" ixy="-0.0011266691" ixz="-0.0000000017"
-				iyy="0.0013220979" iyz="-0.0000000025"
-				izz="0.0053756998"/>
+		<inertia ixx="0.0544481426" ixy="-0.0112666910" ixz="-0.0000000167"
+				iyy="0.0132209786" iyz="-0.0000000248"
+				izz="0.0537569983"/>
 	</inertial>
 </xacro:macro>

File: inertia/F12.xacro (robot description, xacro)
@@ -4,9 +4,9 @@
 <xacro:macro name="foot_inertial">
 	<inertial>
-		<mass value="0.1057487617"/>
+		<mass value="0.0211497523"/>
 		<origin xyz="-0.0019430139 -0.0000550246 -0.0017743149" />
-		<inertia ixx="0.0071021789" ixy="-0.0000021688" ixz="0.0001178392"
-				iyy="0.0179606830" iyz="0.0000017764"
-				izz="0.0247642197"/>
+		<inertia ixx="0.0710217890" ixy="-0.0000216879" ixz="0.0011783916"
+				iyy="0.1796068301" iyz="0.0000177639"
+				izz="0.2476421973"/>
 	</inertial>
 </xacro:macro>

File: inertia/F5.xacro (robot description, xacro)
@@ -4,9 +4,9 @@
 <xacro:macro name="hip_twist_inertial">
 	<inertial>
-		<mass value="0.0755193623"/>
+		<mass value="0.0151038725"/>
 		<origin xyz="0.0005416307 -0.0000009200 0.0190685105" />
-		<inertia ixx="0.0082750315" ixy="-0.0000001051" ixz="0.0002681193"
-				iyy="0.0194814984" iyz="-0.0000005502"
-				izz="0.0133677616"/>
+		<inertia ixx="0.0827503154" ixy="-0.0000010513" ixz="0.0026811928"
+				iyy="0.1948149839" iyz="-0.0000055021"
+				izz="0.1336776164"/>
 	</inertial>
 </xacro:macro>

File: inertia/L_Foot.xacro (robot description, xacro)
@@ -4,9 +4,9 @@
 <xacro:macro name="foot_left_inertial">
 	<inertial>
-		<mass value="0.1867801099"/>
+		<mass value="0.0373560220"/>
 		<origin xyz="-0.0055676472 -0.0035014440 0.0028465215" />
-		<inertia ixx="0.0123437897" ixy="0.0013329200" ixz="-0.0014042040"
-				iyy="0.0351609292" iyz="-0.0011492661"
-				izz="0.0411008628"/>
+		<inertia ixx="0.1234378971" ixy="0.0133291996" ixz="-0.0140420399"
+				iyy="0.3516092920" iyz="-0.0114926614"
+				izz="0.4110086282"/>
 	</inertial>
 </xacro:macro>

File: inertia/L_Tibia.xacro (robot description, xacro)
@@ -4,9 +4,9 @@
 <xacro:macro name="tibia_left_inertial">
 	<inertial>
-		<mass value="0.4326089335"/>
-		<origin xyz="-0.0010052500 0.0002674591 -0.0110862203" />
-		<inertia ixx="0.0541596500" ixy="-0.0001245680" ixz="0.0010887872"
-				iyy="0.0479327482" iyz="-0.0009590411"
-				izz="0.0136097320"/>
+		<mass value="0.0865217867"/>
+		<origin xyz="-0.0010052497 0.0002674591 -0.0110862163" />
+		<inertia ixx="0.5415965019" ixy="-0.0012456852" ixz="0.0108877802"
+				iyy="0.4793274729" iyz="-0.0095904753"
+				izz="0.1360973080"/>
 	</inertial>
 </xacro:macro>

File: inertia/L_hip-R_ankle.xacro (robot description, xacro)
@@ -4,9 +4,9 @@
 <xacro:macro name="ankle_right_inertial">
 	<inertial>
-		<mass value="0.6852429363"/>
-		<origin xyz="0.0183499039 -0.0023512250 -0.0035241953" />
-		<inertia ixx="0.0152904078" ixy="-0.0125481783" ixz="-0.0156374248"
-				iyy="0.1050267499" iyz="0.0020800084"
-				izz="0.1059474294"/>
+		<mass value="0.1370485873"/>
+		<origin xyz="0.0175505223 0.0009625287 -0.0012148213" />
+		<inertia ixx="0.1139696886" ixy="0.0332585730" ixz="-0.0436616116"
+				iyy="0.9538957327" iyz="-0.0004562535"
+				izz="0.9658449360"/>
 	</inertial>
 </xacro:macro>
@@ -14,9 +14,9 @@
 <xacro:macro name="hip_left_inertial">
 	<inertial>
-		<mass value="0.6852429363"/>
-		<origin xyz="0.0183499039 0.0023512250 0.0035241953" />
-		<inertia ixx="0.0152904078" ixy="0.0125481783" ixz="0.0156374248"
-				iyy="0.1050267499" iyz="0.0020800084"
-				izz="0.1059474294"/>
+		<mass value="0.1370485873"/>
+		<origin xyz="0.0175505223 -0.0009625287 0.0012148213" />
+		<inertia ixx="0.1139696886" ixy="-0.0332585730" ixz="0.0436616116"
+				iyy="0.9538957327" iyz="-0.0004562535"
+				izz="0.9658449360"/>
 	</inertial>
 </xacro:macro>

File: inertia/L_lowerarm.xacro (robot description, xacro)
@@ -4,9 +4,9 @@
 <xacro:macro name="lowerarm_left_inertial">
 	<inertial>
-		<mass value="0.3833833954"/>
-		<origin xyz="-0.0009850021 0.0071892817 -0.0005845213" />
-		<inertia ixx="0.0324217403" ixy="-0.0037564102" ixz="0.0000783659"
-				iyy="0.0055165992" iyz="-0.0008307738"
-				izz="0.0307393505"/>
+		<mass value="0.0706166158"/>
+		<origin xyz="-0.0004652630 0.0036453116 -0.0005059590" />
+		<inertia ixx="0.1557970134" ixy="-0.0148826287" ixz="0.0001435379"
+				iyy="0.0418086657" iyz="-0.0039002627"
+				izz="0.1398006125"/>
 	</inertial>
 </xacro:macro>

File: inertia/R_Foot.xacro (robot description, xacro)
@@ -4,9 +4,9 @@
 <xacro:macro name="foot_right_inertial">
 	<inertial>
-		<mass value="0.1867801099"/>
+		<mass value="0.0373560220"/>
 		<origin xyz="-0.0055676472 0.0034398816 0.0028465215" />
-		<inertia ixx="0.0123442309" ixy="-0.0013373380" ixz="-0.0014042040"
-				iyy="0.0351609327" iyz="0.0011525105"
-				izz="0.0411013075"/>
+		<inertia ixx="0.1234423088" ixy="-0.0133733804" ixz="-0.0140420399"
+				iyy="0.3516093267" iyz="0.0115251052"
+				izz="0.4110130747"/>
 	</inertial>
 </xacro:macro>

File: inertia/R_Tibia.xacro (robot description, xacro)
@@ -4,9 +4,9 @@
 <xacro:macro name="tibia_right_inertial">
 	<inertial>
-		<mass value="0.4326089335"/>
-		<origin xyz="-0.0010052500 -0.0012675002 -0.0110864377" />
-		<inertia ixx="0.0542924849" ixy="0.0002115982" ixz="0.0010887655"
-				iyy="0.0479327441" iyz="0.0019185952"
-				izz="0.0137425373"/>
+		<mass value="0.0865217867"/>
+		<origin xyz="-0.0010052497 -0.0012675002 -0.0110864417" />
+		<inertia ixx="0.5429248510" ixy="0.0021159868" ixz="0.0108877466"
+				iyy="0.4793274318" iyz="0.0191858920"
+				izz="0.1374253618"/>
 	</inertial>
 </xacro:macro>

File: inertia/R_hip-L_ankle.xacro (robot description, xacro)
@@ -4,9 +4,9 @@
 <xacro:macro name="ankle_left_inertial">
 	<inertial>
-		<mass value="0.6852429363"/>
-		<origin xyz="0.0167509278 0.0033519500 -0.0035241956" />
-		<inertia ixx="0.0160687475" ixy="0.0135264586" ixz="-0.0142999521"
-				iyy="0.0903445586" iyz="-0.0025649497"
-				izz="0.0920435080"/>
+		<mass value="0.1370485873"/>
+		<origin xyz="0.0175503800 0.0000382013 -0.0012148213" />
+		<inertia ixx="0.1126701697" ixy="-0.0091785729" ixz="-0.0436618956"
+				iyy="0.9538828186" iyz="-0.0012283871"
+				izz="0.9645318393"/>
 	</inertial>
 </xacro:macro>
@@ -14,9 +14,9 @@
 <xacro:macro name="hip_right_inertial">
 	<inertial>
-		<mass value="0.6852429363"/>
-		<origin xyz="0.0167509278 -0.0033519500 0.0035241956" />
-		<inertia ixx="0.0160687475" ixy="-0.0135264586" ixz="0.0142999521"
-				iyy="0.0903445586" iyz="-0.0025649497"
-				izz="0.0920435080"/>
+		<mass value="0.1370485873"/>
+		<origin xyz="0.0175503800 -0.0000382013 0.0012148213" />
+		<inertia ixx="0.1126701697" ixy="0.0091785729" ixz="0.0436618956"
+				iyy="0.9538828186" iyz="-0.0012283871"
+				izz="0.9645318393"/>
 	</inertial>
 </xacro:macro>

File: inertia/R_lowerarm.xacro (robot description, xacro)
@@ -4,9 +4,9 @@
 <xacro:macro name="lowerarm_right_inertial">
 	<inertial>
-		<mass value="0.3833833954"/>
-		<origin xyz="-0.0009848283 -0.0081892817 -0.0005847510" />
-		<inertia ixx="0.0336009689" ixy="0.0038318932" ixz="0.0000784112"
-				iyy="0.0055167096" iyz="0.0008760966"
-				izz="0.0319185839"/>
+		<mass value="0.0706166158"/>
+		<origin xyz="-0.0004650645 -0.0046453116 -0.0005062069" />
+		<inertia ixx="0.1616520824" ixy="0.0152109261" ixz="0.0001440817"
+				iyy="0.0418097664" iyz="0.0042626086"
+				izz="0.1456557322"/>
 	</inertial>
 </xacro:macro>

File: inertia/Torso.xacro (robot description, xacro)
@@ -4,9 +4,9 @@
 <xacro:macro name="torso_inertial">
 	<inertial>
-		<mass value="3.4770266466"/>
-		<origin xyz="0.0162019036 0.0049844800 0.0038595353" />
-		<inertia ixx="0.9787053684" ixy="0.0543464614" ixz="-0.0262073548"
-				iyy="0.9730952674" iyz="0.0198675713"
-				izz="0.9352573858"/>
+		<mass value="0.6954053293"/>
+		<origin xyz="0.0171121538 0.0052995599 0.0016431550" />
+		<inertia ixx="10.9003247826" ixy="0.7020020095" ixz="-1.0245344637"
+				iyy="10.6912796312" iyz="0.0302048573"
+				izz="10.3158095391"/>
 	</inertial>
 </xacro:macro>

File: inertia/upperarm.xacro (robot description, xacro)
@@ -4,9 +4,9 @@
 <xacro:macro name="upperarm_right_inertial">
 	<inertial>
-		<mass value="0.3822870734"/>
-		<origin xyz="-0.0000002032 -0.0068291604 -0.0006710552" />
-		<inertia ixx="0.0274690892" ixy="0.0000004066" ixz="-0.0000000859"
-				iyy="0.0077817002" iyz="0.0007139012"
-				izz="0.0226034759"/>
+		<mass value="0.0764574147"/>
+		<origin xyz="-0.0000001987 -0.0068291607 -0.0006710552" />
+		<inertia ixx="0.2746908812" ixy="0.0000041559" ixz="-0.0000007966"
+				iyy="0.0778170043" iyz="0.0071390070"
+				izz="0.2260347501"/>
 	</inertial>
 </xacro:macro>
@@ -14,9 +14,9 @@
 <xacro:macro name="upperarm_left_inertial">
 	<inertial>
-		<mass value="0.3822870734"/>
-		<origin xyz="0.0000002032 0.0068291604 -0.0006710552" />
-		<inertia ixx="0.0274690892" ixy="0.0000004066" ixz="0.0000000859"
-				iyy="0.0077817002" iyz="-0.0007139012"
-				izz="0.0226034759"/>
+		<mass value="0.0764574147"/>
+		<origin xyz="0.0000001987 0.0068291607 -0.0006710552" />
+		<inertia ixx="0.2746908812" ixy="0.0000041559" ixz="0.0000007966"
+				iyy="0.0778170043" iyz="-0.0071390070"
+				izz="0.2260347501"/>
 	</inertial>
 </xacro:macro>

File: inertia/upperleg.xacro (robot description, xacro)
@@ -4,9 +4,9 @@
 <xacro:macro name="upperleg_inertial">
 	<inertial>
-		<mass value="0.1557654222"/>
+		<mass value="0.0311530844"/>
 		<origin xyz="-0.0012110096 0.0000000568 -0.0444074895" />
-		<inertia ixx="0.0867975538" ixy="-0.0000000255" ixz="0.0030686267"
-				iyy="0.0784005596" iyz="-0.0000000875"
-				izz="0.0138679533"/>
+		<inertia ixx="0.8679755381" ixy="-0.0000002549" ixz="0.0306862669"
+				iyy="0.7840055957" iyz="-0.0000008749"
+				izz="0.1386795334"/>
 	</inertial>
 </xacro:macro>

File: typea.urdf (robot description, URDF)
Before this commit: robot typea, 25 links, 24 joints
Links:
- link imu_link: mass 0.001 -> None; geometry visual box size=0.04 0.02 0.005
- link l_ankle_lateral_link: mass 0.1867801099 -> 0.0373560220; geometry collision box size=0.0405 0.029 0.083; visual mesh filename=file:///home/matthew/catkin_ws/src/bioloid_typea_descriptio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 scale=0.001 0.001 0.001
- link l_ankle_swing_link: mass 0.6852429363 -> 0.1370485873; geometry collision box size=0.051 0.0721 0.04; visual mesh filename=file:///home/matthew/catkin_ws/src/bioloid_typea_descriptio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 scale=0.001 0.001 0.001
- link l_foot_link: mass 0.1867801099 -> 0.0373560220; geometry collision box size=0.009 0.061 0.101; visual mesh filename=file:///home/matthew/catkin_ws/src/bioloid_typea_descriptio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 scale=0.001 0.001 0.001
- link l_hand_link: mass 0.0303003163 -> 0.0060600633; geometry collision box size=0.0131 0.0265 0.044; collision box size=0.0575 0.0175 0.035
- link l_hip_lateral_link: mass 0.6852429363 -> 0.1370485873; geometry collision box size=0.04 0.051 0.0721; visual mesh filename=file:///home/matthew/catkin_ws/src/bioloid_typea_descriptio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 scale=0.001 0.001 0.001
- link l_hip_twist_link: mass 0.0755193623 -> 0.0151038725; geometry collision box size=0.029 0.083 0.0405; visual mesh filename=file:///home/matthew/catkin_ws/src/bioloid_typea_descriptio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 scale=0.001 0.001 0.001
- link l_lower_arm_link: mass 0.3822870734 -> 0.0764574147; geometry collision box size=0.058 0.033 0.044; visual mesh filename=file:///home/matthew/catkin_ws/src/bioloid_typea_descriptio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 scale=0.001 0.001 0.001
- link l_lower_leg_link: mass 0.4326089335 -> 0.0865217867; geometry collision box size=0.033 0.051 0.044; collision box size=0.067 0.03 0.049
- link l_shoulder_swing_link: mass 0.0595945816 -> 0.0119189163; geometry collision box size=0.052 0.039 0.036; visual mesh filename=file:///home/matthew/catkin_ws/src/bioloid_typea_descriptio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 scale=0.001 0.001 0.001
- link l_upper_arm_link: mass 0.3822870734 -> 0.0764574147; geometry collision box size=0.047 0.033 0.052; collision box size=0.054 0.033 0.044
- link l_upper_leg_link: mass 0.1557654222 -> 0.0311530844; geometry collision box size=0.04 0.0371 0.049; collision box size=0.065 0.03 0.049
- link r_ankle_lateral_link: mass 0.1867801099 -> 0.0373560220; geometry collision box size=0.0405 0.029 0.083; visual mesh filename=file:///home/matthew/catkin_ws/src/bioloid_typea_descriptio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 scale=0.001 0.001 0.001
- link r_ankle_swing_link: mass 0.6852429363 -> 0.1370485873; geometry collision box size=0.051 0.0721 0.04; visual mesh filename=file:///home/matthew/catkin_ws/src/bioloid_typea_descriptio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 scale=0.001 0.001 0.001
- link r_foot_link: mass 0.1867801099 -> 0.0373560220; geometry collision box size=0.009 0.061 0.101; visual mesh filename=file:///home/matthew/catkin_ws/src/bioloid_typea_descriptio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 scale=0.001 0.001 0.001
- link r_hand_link: mass 0.0303003163 -> 0.0060600633; geometry collision box size=0.0131 0.0265 0.044; collision box size=0.0575 0.0175 0.035
- link r_hip_lateral_link: mass 0.6852429363 -> 0.1370485873; geometry collision box size=0.04 0.051 0.0721; visual mesh filename=file:///home/matthew/catkin_ws/src/bioloid_typea_descriptio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 scale=0.001 0.001 0.001
- link r_hip_twist_link: mass 0.0755193623 -> 0.0151038725; geometry collision box size=0.029 0.083 0.0405; visual mesh filename=file:///home/matthew/catkin_ws/src/bioloid_typea_descriptio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 scale=0.001 0.001 0.001
- link r_lower_arm_link: mass 0.3833833954 -> 0.0706166158; geometry collision box size=0.058 0.033 0.044; visual mesh filename=file:///home/matthew/catkin_ws/src/bioloid_typea_descriptio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 scale=0.001 0.001 0.001
- link r_lower_leg_link: mass 0.4326089335 -> 0.0865217867; geometry collision box size=0.033 0.051 0.044; collision box size=0.067 0.03 0.049
- link r_shoulder_swing_link: mass 0.0595945816 -> 0.0119189163; geometry collision box size=0.052 0.039 0.036; visual mesh filename=file:///home/matthew/catkin_ws/src/bioloid_typea_descriptio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 scale=0.001 0.001 0.001
- link r_upper_arm_link: mass 0.3822870734 -> 0.0764574147; geometry collision box size=0.047 0.033 0.052; collision box size=0.054 0.033 0.044
- link r_upper_leg_link: mass 0.1557654222 -> 0.0311530844; geometry collision box size=0.04 0.0371 0.049; collision box size=0.065 0.03 0.049
- link torso_link: mass 3.4770266466 -> 0.6954053293; geometry collision box size=0.054 0.033 0.044; collision box size=0.065 0.099 0.043
Joints:
- joint imu_to_base_joint: axis 1 0 0 -> (none); child imu_link -> base_link; origin xyz=0 0 0.05 rpy=0 0 0 -> xyz=0.01 0 0.0788 rpy=0 0 0; parent base_link -> imu_link
- joint l_ankle_lateral_joint: axis 0 0 1 -> 0 0 -1; limit lower=-0.8 upper=0.8 effort=10 velocity=5.6548668 -> lower=-0.5 upper=0.5 effort=10 velocity=5.6548668; origin xyz=0 0 0 rpy=-1.57079632679 0 0 -> xyz=0 0 0 rpy=-1.570795 0 0
- joint l_ankle_swing_joint: origin xyz=-0.071 -0.0145 0 rpy=3.14159265359 0 0 -> xyz=-0.071 -0.0145 0 rpy=3.14159 0 0
- joint l_elbow_joint: axis 0 0 1 -> 0 0 1.0
- joint l_hip_lateral_joint: axis 0 0 1 -> 0 0 -1; limit lower=-0.8 upper=0.8 effort=10 velocity=5.6548668 -> lower=-0.6 upper=0.6 effort=10 velocity=5.6548668; origin xyz=0 0 0.05 rpy=1.57079632679 0 0 -> xyz=0 0 0.05 rpy=1.570795 0 0
- joint l_hip_swing_joint: origin xyz=0 0 0 rpy=1.57079632679 0 -1.57079632679 -> xyz=0 0 0 rpy=1.570795 0 -1.570795
- joint l_hip_twist_joint: origin xyz=0 0.0385 -0.0655 rpy=0 3.14159265359 -1.57079632679 -> xyz=0 0.0385 -0.0655 rpy=0 3.14159 -1.570795
- joint l_knee_joint: axis 0 0 1 -> 0 0 -1; limit lower=-2 upper=0 effort=10 velocity=5.6548668 -> lower=0.0 upper=2.0 effort=10 velocity=5.6548668
- joint l_shoulder_lateral_joint: axis 0 0 1 -> 0 0 1.0; origin xyz=0 0.014 0.044 rpy=0 -1.57079632679 0 -> xyz=0 0.014 0.044 rpy=0 -1.570795 0
- joint l_shoulder_swing_joint: limit lower=-1 upper=1.57079632679 effort=2.8 velocity=1.0 -> lower=-1.570795 upper=1.570795 effort=2.8 velocity=1.0; origin xyz=0 0.032 0 rpy=-1.57079632679 -1.57079632679 0 -> xyz=0 0.032 0 rpy=-1.570795 -1.570795 0
- joint r_ankle_lateral_joint: axis 0 0 1 -> 0 0 -1; limit lower=-0.8 upper=0.8 effort=10 velocity=5.6548668 -> lower=-0.5 upper=0.5 effort=10 velocity=5.6548668; origin xyz=0 0 0 rpy=-1.57079632679 0 0 -> xyz=0 0 0 rpy=-1.570795 0 0
- joint r_ankle_swing_joint: origin xyz=0.071 -0.0145 0 rpy=3.14159265359 0 0 -> xyz=0.071 -0.0145 0 rpy=3.14159 0 0
- joint r_elbow_joint: axis 0 0 1 -> 0 0 -1.0
- joint r_hip_lateral_joint: axis 0 0 1 -> 0 0 -1; limit lower=-0.8 upper=0.8 effort=10 velocity=5.6548668 -> lower=-0.6 upper=0.6 effort=10 velocity=5.6548668; origin xyz=0 0 0.05 rpy=-1.57079632679 0 0 -> xyz=0 0 0.05 rpy=-1.570795 0 0
- joint r_hip_swing_joint: origin xyz=0 0 0 rpy=1.57079632679 0 -1.57079632679 -> xyz=0 0 0 rpy=1.570795 0 -1.570795
- joint r_hip_twist_joint: origin xyz=0 -0.0385 -0.0655 rpy=0 3.14159265359 1.57079632679 -> xyz=0 -0.0385 -0.0655 rpy=0 3.14159 1.570795
- joint r_knee_joint: axis 0 0 1 -> 0 0 -1; limit lower=0 upper=2 effort=10 velocity=5.6548668 -> lower=-2.0 upper=0.0 effort=10 velocity=5.6548668
- joint r_shoulder_lateral_joint: axis 0 0 1 -> 0 0 -1.0; origin xyz=0 0.014 0.044 rpy=0 -1.57079632679 0 -> xyz=0 0.014 0.044 rpy=0 -1.570795 0
- joint r_shoulder_swing_joint: limit lower=-1 upper=1.57079632679 effort=2.8 velocity=1.0 -> lower=-1.570795 upper=1.570795 effort=2.8 velocity=1.0; origin xyz=0 -0.032 0 rpy=1.57079632679 1.57079632679 0 -> xyz=0 -0.032 0 rpy=1.570795 1.570795 0
