Commit message: Add files via upload

File: typea.xacro (robot description, xacro)
@@ -19,5 +19,5 @@
     <!-- Import gazebo_ros_control plugin -->
     <xacro:include filename="$(find bioloid_typea_description)/gazebo.xacro" ns="gazebo"/>
-    <!--  <xacro:property name="pi" value="3.14159"/> -->
+    <xacro:property name="pi" value="3.14159"/>
     <xacro:property name="cad_dir" value="file://$(find bioloid_typea_description)/assets/cad"/>
     <!-- Typically, STL/DAE model units are in mm, but RViz units are in m, hence models must be scaled down by 1000. -->
@@ -36,12 +36,10 @@
     <!-- IMU -->
     <joint name="imu_to_base_joint" type="fixed">
-        <axis xyz="1 0 0"/>
-        <origin xyz="0 0 0.05" rpy="0 0 0"/>
-        <parent link="base_link"/>
-        <child link="imu_link"/>
+        <parent link="imu_link"/>
+        <origin xyz="0.01 0 0.0788" rpy="0 0 0"/>
+        <child link="base_link"/>
     </joint>
     <link name="imu_link">
         <visual>
-            <origin rpy="0 0 0" xyz="0 0 0"/>
             <geometry>
                 <box size="0.04 0.02 0.005"/>
@@ -51,15 +49,9 @@
             </material>
         </visual>
-          <collision>
-	    <origin rpy="0 0 0" xyz="0 0 0"/>
-	        <geometry>
-	        <box size=".01 .01 .01"/>
-	        </geometry>
-	    </collision>
-	  <inertial>
-	    <mass value="0.001"/>
-	    <origin rpy="0 0 0" xyz="0 0 0"/>
-	    <inertia ixx="0.0001" ixy="0" ixz="0" iyy="0.000001" iyz="0" izz="0.0001"/>
-	  </inertial>
+        <!--<inertial>
+            <origin xyz="0 0 0"/>
+            <mass value="1.0"/>
+            <inertia  ixx="0.001" ixy="0.0"  ixz="0.0"  iyy="0.001"  iyz="0.0"  izz="0.001"/>
+        </inertial>-->
     </link>
     <xacro:macro name="shoulder_swing_joint" params="prefix reflect">
@@ -69,5 +61,5 @@
             <xacro:z_rot/>
             <child link="${prefix}_shoulder_swing_link"/>
-            <limit lower="-1" upper="${pi/2}" effort="2.8" velocity="1.0"/>
+            <limit lower="${-pi/2}" upper="${pi/2}" effort="2.8" velocity="1.0"/>
         </joint>
     </xacro:macro>
@@ -76,5 +68,5 @@
             <parent link="${prefix}_shoulder_swing_link"/>
             <origin xyz="0 0.014 0.044" rpy="0 ${-pi/2} 0"/>
-            <xacro:z_rot/>
+            <axis xyz="0 0 ${reflect*-1}"/>
             <child link="${prefix}_upper_arm_link"/>
             <limit lower="-1.5" upper="1.5" effort="2.8" velocity="1.0"/>
@@ -85,5 +77,5 @@
             <parent link="${prefix}_upper_arm_link"/>
             <origin xyz="0.0675 0 0" rpy="0 0 0"/>
-            <xacro:z_rot/>
+            <axis xyz="0 0 ${reflect*-1}"/>
             <child link="${prefix}_lower_arm_link"/>
             <limit lower="-1.77" upper="1.77" effort="2.8" velocity="1.0"/>
@@ -109,8 +101,8 @@
         <joint name="${prefix}_hip_lateral_joint" type="revolute">
             <parent link="${prefix}_hip_twist_link"/>
-            <origin xyz="0 0 0.05" rpy="${reflect*-pi/2} 0 0"/>
-            <xacro:z_rot/>
+            <origin xyz="0 0 0.05" rpy="${reflect*pi/2} 0 0"/>
+            <axis xyz="0 0 -1"/>
             <child link="${prefix}_hip_lateral_link"/>
-            <limit lower="-0.8" upper="0.8" effort="10" velocity="5.6548668"/>
+            <limit lower="-0.6" upper="0.6" effort="10" velocity="5.6548668"/>
         </joint>
     </xacro:macro>
@@ -127,6 +119,6 @@
         <joint name="${prefix}_knee_joint" type="revolute">
             <parent link="${prefix}_upper_leg_link"/>
-            <origin xyz="${reflect*0.075} 0.0145 0" rpy="0 0 0"/>
-            <axis xyz="0 0 1"/>
+            <origin xyz="${reflect*-0.075} 0.0145 0" rpy="0 0 0"/>
+            <axis xyz="0 0 -1"/>
             <child link="${prefix}_lower_leg_link"/>
             <limit lower="${-1+reflect}" upper="${1+reflect}" effort="10" velocity="5.6548668"/>
@@ -146,7 +138,7 @@
             <parent link="${prefix}_ankle_swing_link"/>
             <origin xyz="0 0 0" rpy="${-pi/2} 0 0"/>
-            <xacro:z_rot/>
+            <axis xyz="0 0 -1"/>
             <child link="${prefix}_ankle_lateral_link"/>
-            <limit lower="-0.8" upper="0.8" effort="10" velocity="5.6548668"/>
+            <limit lower="-0.5" upper="0.5" effort="10" velocity="5.6548668"/>
         </joint>
     </xacro:macro>
@@ -641,10 +633,10 @@
     <xacro:hip_twist_link prefix="l" reflect="-1" x_offset="0" y_offset="0.02" z_offset="0"/>
     <!-- Right hip twist to hip lateral -->
-    <xacro:hip_lateral_joint prefix="r" reflect="1"/>
+    <xacro:hip_lateral_joint prefix="r" reflect="-1"/>
     <xacro:hip_lateral_link prefix="r" reflect="1" x_offset="0" y_offset="0" z_offset="0.0353">
     	<xacro:hip_right_inertial/>
     </xacro:hip_lateral_link>
     <!-- Left hip twist to hip lateral -->
-    <xacro:hip_lateral_joint prefix="l" reflect="-1"/>
+    <xacro:hip_lateral_joint prefix="l" reflect="1"/>
     <xacro:hip_lateral_link prefix="l" reflect="-1" x_offset="0" y_offset="0" z_offset="0.0353">
 		<xacro:hip_left_inertial/>
@@ -657,10 +649,10 @@
     <xacro:upper_leg_link prefix="l" reflect="-1" x_offset="0" y_offset="0" z_offset="0"/>
     <!-- Right upper leg to lower leg -->
-    <xacro:knee_joint prefix="r" reflect="1"/>
+    <xacro:knee_joint prefix="r" reflect="-1"/>
     <xacro:lower_leg_link prefix="r" reflect="1" x_offset="0" y_offset="0" z_offset="0">
     	<xacro:tibia_right_inertial/>
     </xacro:lower_leg_link>
     <!-- Left upper leg to lower leg -->
-    <xacro:knee_joint prefix="l" reflect="-1"/>
+    <xacro:knee_joint prefix="l" reflect="1"/>
     <xacro:lower_leg_link prefix="l" reflect="-1" x_offset="0" y_offset="0" z_offset="0">
     	<xacro:tibia_left_inertial/>
